File: LED_RAM/LED_RAM.kicad_sch (KiCad schematic)
At the start: 80 parts, among them J1 GND, J10 USB_C_Receptacle_PowerOnly_6P, J13 Conn_01x22_Pin, J14 Conn_01x22_Pin, J15 Conn_01x22_Pin, J16 Conn_01x22_Pin, J2 5V, J3 DOUT, J4 DIN, J7 DIN, J8 GND, J9 5V, U1 ER_OLEDM0.91_1x-I2C, U2 ER_OLEDM0.91_1x-I2C

Commit message: Add files via upload
Parts:
- removed J1: GND, symbol Connector:Conn_01x01_Pin
- added J12: Conn_01x08_Pin, Connector_PinHeader_2.54mm:PinHeader_1x08_P2.54mm_Vertical, symbol Connector:Conn_01x08_Pin
- added J3: GND, Connector_PinHeader_2.54mm:PinHeader_1x01_P2.54mm_Vertical, symbol Connector:Conn_01x01_Pin
- added J5: Conn_01x05_Pin, Connector_PinHeader_2.54mm:PinHeader_1x05_P2.54mm_Vertical, symbol Connector:Conn_01x05_Pin
- added J6: Conn_01x10_Pin, Connector_PinHeader_2.54mm:PinHeader_1x10_P2.54mm_Vertical, symbol Connector:Conn_01x10_Pin
- added U3: (no value), PCM_Package_DIP_AKL:DIP-48_W15.24mm, symbol cy7c130:cy7c130
- added U5, U6, U7: TXS0108EPW, Package_SO:TSSOP-20_4.4x6.5mm_P0.65mm, symbol Logic_LevelTranslator:TXS0108EPW
- J1: renamed from J4; footprint (none) -> Connector_PinHeader_2.54mm:PinHeader_1x01_P2.54mm_Vertical
- J10: footprint (none) -> Connector_USB:USB_C_Receptacle_GCT_USB4125-xx-x_6P_TopMnt_Horizontal
- J2, J7, J8, J9: footprint (none) -> Connector_PinHeader_2.54mm:PinHeader_1x01_P2.54mm_Vertical
- J4: renamed from J3; footprint (none) -> Connector_PinHeader_2.54mm:PinHeader_1x01_P2.54mm_Vertical
- R1, R2: footprint (none) -> Resistor_THT:R_Axial_DIN0207_L6.3mm_D2.5mm_P7.62mm_Horizontal
- renumbered D19 to D18, D21 to D19, D23 to D20, D25 to D21, D27 to D22, D29 to D23, D31 to D24, D18 to D25, D20 to D26, D22 to D27, D24 to D28, D26 to D29, D28 to D30, D30 to D31, D37 to D34, D41 to D35, D45 to D36, D49 to D37, D53 to D38, D57 to D39, D61 to D40, D34 to D41, D38 to D42, D42 to D43, D46 to D44, D50 to D45, D54 to D46, D58 to D47, D62 to D48, D35 to D49, D39 to D50, D43 to D51, D47 to D52, D51 to D53, D55 to D54, D59 to D55, D63 to D56, D36 to D57, D40 to D58, D44 to D59, D48 to D60, D52 to D61, D56 to D62, D60 to D63
Connections:
- net GND: now also J10.A12 (GND), J10.B12 (GND), J10.SH (SHIELD), J8.1 (Pin_1), R1.1, R2.1, U1.1 (GND), U2.1 (GND), J3.1 (Pin_1), U3.24 (GND), U5.11 (GND), U6.11 (GND), U7.11 (GND)
- net 3.3v: now reaches J15.1 (Pin_1), J16.1 (Pin_1)
- net 3.3v: now also U1.2 (VCC), U2.2 (VCC), U5.10 (OE), U5.2 (VCCA), U6.10 (OE), U6.2 (VCCA), U7.10 (OE), U7.2 (VCCA)
- net IO0_L: now reaches J15.10 (Pin_10), J16.10 (Pin_10)
- net IO0_L: now also U7.1 (A1)
- net IO1_L: now reaches J15.11 (Pin_11), J16.11 (Pin_11)
- net IO1_L: now also U7.3 (A2)
- net A1_L: now reaches J15.12 (Pin_12), J16.12 (Pin_12)
- net A1_L: now also U5.8 (A7)
- net SCL: now reaches J15.14 (Pin_14), J16.14 (Pin_14)
- net SCL: now also U1.3 (SCL), U2.3 (SCL)
- net A2_L: now reaches J15.15 (Pin_15), J16.15 (Pin_15)
- net A2_L: now also U5.9 (A8)
- net A3_L: now reaches J15.16 (Pin_16), J16.16 (Pin_16)
- net A3_L: now also U6.1 (A1)
- net A4_L: now reaches J15.17 (Pin_17), J16.17 (Pin_17)
- net A4_L: now also U6.3 (A2)
- net A5_L: now reaches J15.18 (Pin_18), J16.18 (Pin_18)
- net A5_L: now also U6.4 (A3)
- net A6_L: now reaches J15.19 (Pin_19), J16.19 (Pin_19)
- net A6_L: now also U6.5 (A4)
- net A7_L: now reaches J15.20 (Pin_20), J16.20 (Pin_20)
- net A7_L: now also U6.6 (A5)
- net 5V: now reaches J15.21 (Pin_21), J16.21 (Pin_21)
- net 5V: now also J10.A9 (VBUS), J10.B9 (VBUS), J9.1 (Pin_1), U3.48 (VCC), U5.19 (VCCB), U6.19 (VCCB), U7.19 (VCCB)
- net ~{BUSY_L}: now reaches J15.4 (Pin_4), J16.4 (Pin_4)
- net ~{BUSY_L}: now also U5.4 (A3)
- net ~{INT_L}: now reaches J15.5 (Pin_5), J16.5 (Pin_5)
- net ~{INT_L}: now also U5.5 (A4)
- net ~{OE_L}: now reaches J15.6 (Pin_6), J16.6 (Pin_6)
- net ~{OE_L}: now also U5.6 (A5)
- net A0_L: now reaches J15.7 (Pin_7), J16.7 (Pin_7)
- net A0_L: now also U5.7 (A6)
- net A8_L: now reaches J15.8 (Pin_8), J16.8 (Pin_8)
- net A8_L: now also U6.7 (A6)
- net A9_L: now reaches J15.9 (Pin_9), J16.9 (Pin_9)
- net A9_L: now also U6.8 (A7)
- net IO2_L: now reaches J13.13 (Pin_13), J14.13 (Pin_13)
- net IO2_L: now also U7.4 (A3)
- net IO3_L: now reaches J13.14 (Pin_14), J14.14 (Pin_14)
- net IO3_L: now also U7.5 (A4)
- net IO4_L: now reaches J13.15 (Pin_15), J14.15 (Pin_15)
- net IO4_L: now also U7.6 (A5)
- net IO5_L: now reaches J13.16 (Pin_16), J14.16 (Pin_16)
- net IO5_L: now also U7.7 (A6)
- net IO6_L: now reaches J13.17 (Pin_17), J14.17 (Pin_17)
- net IO6_L: now also U7.8 (A7)
- net ~{RW_L}: now reaches J13.18 (Pin_18), J14.18 (Pin_18)
- net ~{RW_L}: now also U5.3 (A2)
- net ~{CE_L}: now reaches J13.19 (Pin_19), J14.19 (Pin_19)
- net ~{CE_L}: now also U5.1 (A1)
- net IO7_L: now reaches J13.6 (Pin_6), J14.6 (Pin_6)
- net IO7_L: now also U7.9 (A8)
- net at J13.7 (Pin_7), J14.7 (Pin_7): now also J7.1 (Pin_1)
- net SDA: now reaches J13.8 (Pin_8), J14.8 (Pin_8)
- net SDA: now also U1.4 (SDA), U2.4 (SDA)
- new net: U3.1 (~{CE_L}), U5.20 (B1)
- new net: U3.10 (A4_L), U6.18 (B2)
- new net: U3.11 (A5_L), U6.17 (B3)
- new net: U3.12 (A6_L), U6.16 (B4)
- new net: U3.13 (A7_L), U6.15 (B5)
- new net: U3.14 (A8_L), U6.14 (B6)
- new net: U3.15 (A9_L), U6.13 (B7)
- new net: U3.16 (IO0_L), U7.20 (B1)
- new net: U3.17 (IO1_L), U7.18 (B2)
- new net: U3.18 (IO2_L), U7.17 (B3)
- new net: U3.19 (IO3_L), U7.16 (B4)
- new net: U3.2 (~{RW_L}), U5.18 (B2)
- new net: U3.20 (IO4_L), U7.15 (B5)
- new net: U3.21 (IO5_L), U7.14 (B6)
- new net: U3.22 (IO6_L), U7.13 (B7)
- new net: U3.23 (IO7_L), U7.12 (B8)
- new net: J12.1 (Pin_1), U3.25 (IO7_R)
- new net: J12.2 (Pin_2), U3.26 (IO6_R)
- new net: J12.3 (Pin_3), U3.27 (IO5_R)
- new net: J12.4 (Pin_4), U3.28 (IO4_R)
- new net: J12.5 (Pin_5), U3.29 (IO3_R)
- new net: U3.3 (~{BUSY_L}), U5.17 (B3)
- new net: J12.6 (Pin_6), U3.30 (IO2_R)
- new net: J12.7 (Pin_7), U3.31 (IO1_R)
- new net: J12.8 (Pin_8), U3.32 (IO0_R)
- new net: J6.1 (Pin_1), U3.33 (A9_R)
- new net: J6.2 (Pin_2), U3.34 (A8_R)
- new net: J6.3 (Pin_3), U3.35 (A7_R)
- new net: J6.4 (Pin_4), U3.36 (A6_R)
- new net: J6.5 (Pin_5), U3.37 (A5_R)
- new net: J6.6 (Pin_6), U3.38 (A4_R)
- new net: J6.7 (Pin_7), U3.39 (A3_R)
- new net: U3.4 (~{INT_L}), U5.16 (B4)
- new net: J6.8 (Pin_8), U3.40 (A2_R)
- new net: J6.9 (Pin_9), U3.41 (A1_R)
- new net: J6.10 (Pin_10), U3.42 (A0_R)
- new net: J5.1 (Pin_1), U3.43 (~{OE_R})
- new net: J5.2 (Pin_2), U3.44 (~{INT_R})
- new net: J5.3 (Pin_3), U3.45 (~{BUSY_R})
- new net: J5.4 (Pin_4), U3.46 (~{RW_R})
- new net: J5.5 (Pin_5), U3.47 (~{CE_R})
- new net: U3.5 (~{OE_L}), U5.15 (B5)
- new net: U3.6 (A0_L), U5.14 (B6)
- new net: U3.7 (A1_L), U5.13 (B7)
- new net: U3.8 (A2_L), U5.12 (B8)
- new net: U3.9 (A3_L), U6.20 (B1)
Other:
- note added: "1, 2, 4, 5, 6, 7, 8, 9, 10, 11, 12, 13, 14, 15, 16, 17, 18, 38, 39, 40, 41, 42, 47"
- moved on the sheet: U1, U2
