File: LED_RAM/LED_RAM.kicad_pcb (KiCad board)
At the start: 2 copper layers, 190.4 x 184.2 mm, 89 parts, among them J1 DIN, J10 USB_C_Receptacle_PowerOnly_6P, J12 Conn_01x08_Pin, J13 Conn_01x22_Pin, J14 Conn_01x22_Pin, J15 Conn_01x22_Pin, J16 Conn_01x22_Pin, J2 5V, J3 GND, J4 DOUT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

Commit message: Add files via upload
Parts:
- added ?: , , F.Cu at (70.4, 24.0)
- added J9: 5V, Connector_PinHeader_2.54mm:PinHeader_1x01_P2.54mm_Vertical, F.Cu at (255.4, 23.8)
- moved D3 323.3 mm to (70.7, -130.8)
- moved J3 323.3 mm to (65.7, -5.62)
- moved D1 323.3 mm to (70.8, -180.7)
- moved D10 323.3 mm to (95.4, -155.9)
- moved D11 323.3 mm to (95.4, -130.9)
- moved D12 323.3 mm to (95.4, -105.9)
- moved D13 323.3 mm to (95.4, -80.9)
- moved D14 323.3 mm to (95.4, -55.9)
- moved D15 323.3 mm to (95.4, -30.9)
- moved D16 323.3 mm to (95.4, -5.88)
- moved D17 323.3 mm to (120.6, -180.9)
- moved D18 323.3 mm to (120.6, -155.9)
- moved D19 323.3 mm to (120.6, -130.9)
- moved D2 323.3 mm to (70.8, -155.9)
- moved D20 323.3 mm to (120.6, -105.9)
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Routing:
- net /5V: track 0.00 -> 245.7 mm, vias 0 -> 3
- net GND: track 1624.2 -> 1839.1 mm
- net /SDA: track 0.00 -> 196.4 mm
- net /3.3v: track 0.00 -> 196.4 mm
- net /SCL: track 0.00 -> 186.9 mm
- net Net-(J13-Pin_7): track 0.00 -> 160.3 mm
- net /~{CE_L}: track 0.00 -> 73.4 mm
- net /IO2_L: track 0.00 -> 54.8 mm
- net /IO3_L: track 0.00 -> 54.0 mm
- net /IO4_L: track 0.00 -> 53.2 mm
- net /IO6_L: track 0.00 -> 52.7 mm
- net /IO5_L: track 0.00 -> 52.5 mm
- net Net-(U3-~{CE_L}): track 0.00 -> 29.9 mm
- net Net-(U3-~{RW_L}): track 0.00 -> 28.2 mm
- net Net-(U3-~{BUSY_L}): track 0.00 -> 26.3 mm
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Other:
- board size 190.4 x 184.2 mm -> 196.3 x 403.9 mm

Commit message: Add files via upload
Routing:
- net GND: track 1839.1 -> 2091.1 mm
- net /IO7_L: track 4.59 -> 91.7 mm
- net /~{RW_L}: track 4.59 -> 88.6 mm, vias 0 -> 1
- net /~{BUSY_L}: track 4.59 -> 49.9 mm, vias 0 -> 2
- net /~{INT_L}: track 4.59 -> 46.7 mm, vias 0 -> 2
- net /A7_L: track 4.59 -> 44.6 mm, vias 0 -> 2
- net /~{OE_L}: track 4.59 -> 43.7 mm, vias 0 -> 2
- net /A6_L: track 4.59 -> 41.3 mm, vias 0 -> 2
- net /A0_L: track 4.59 -> 40.5 mm, vias 0 -> 2
- net /A5_L: track 4.59 -> 39.0 mm, vias 0 -> 2
- net /A4_L: track 4.59 -> 35.9 mm, vias 0 -> 2
- net /A8_L: track 4.59 -> 30.8 mm, vias 0 -> 2
- net /A3_L: track 4.59 -> 29.4 mm, vias 0 -> 2
- net /A9_L: track 4.59 -> 28.9 mm, vias 0 -> 2
- net /A2_L: track 4.59 -> 25.2 mm, vias 0 -> 2
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
Commit message: Add files via upload
Parts:
- moved D33 290.1 mm to (-33.7, 25.3)
- moved D34 290.1 mm to (-33.7, 50.3)
- moved D35 290.1 mm to (-33.7, 75.3)
- moved D38 290.1 mm to (-33.7, 150.3)
- moved D39 290.1 mm to (-33.7, 175.3)
- moved D40 290.1 mm to (-33.7, 200.3)
- moved J1 290.1 mm to (-46.9, 204.6)
- moved J2 290.1 mm to (46.3, 25.1)
- moved J4 290.1 mm to (-50.5, 204.6)
- moved D1 290.1 mm to (-133.4, 25.2)
- moved D10 290.1 mm to (-108.9, 50.1)
- moved D11 290.1 mm to (-108.9, 75.1)
- moved D12 290.1 mm to (-108.9, 100.1)
- moved D13 290.1 mm to (-108.9, 125.1)
- moved D14 290.1 mm to (-108.9, 150.1)
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Other:
- board size 196.3 x 403.9 mm -> 400.6 x 200.2 mm
- board text added: "SOUP-A COOL LED CUBE :D for FallOut 2026"

Commit message: Add files via upload
Parts:
- moved J9 55.9 mm to (255.0, 79.8)
- moved ? 55.9 mm to (70.0, 80.0)
- moved J9 43.5 mm to (255.0, 155.4)
- moved U3 43.5 mm to (245.4, 150.3)
- moved J15 43.5 mm to (187.6, 112.4)
- moved J16 43.5 mm to (187.6, 107.8)
- moved J10 43.5 mm to (255.2, 138.7)
- moved J12 43.5 mm to (184.5, 172.6)
- moved J13 43.5 mm to (240.9, 80.3)
- moved J14 43.5 mm to (240.9, 84.9)
- moved J5 43.5 mm to (232.2, 172.6)
- moved J6 43.5 mm to (205.8, 172.6)
- moved J7 43.5 mm to (161.7, 159.8)
- moved J8 43.5 mm to (70.0, 155.6)
- moved R1 43.5 mm to (240.5, 137.0)
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Routing:
- net /5V: track 245.7 -> 146.3 mm
- net GND: track 2091.1 -> 1991.8 mm
- net Net-(J13-Pin_7): track 160.3 -> 149.0 mm
Other:
- board size 400.6 x 200.2 mm -> 400.1 x 184.2 mm
